File: brd/main_v0.3_simple/RdL_main_v03_simple.brd (EAGLE design)
At the start: 48 x 31.1 mm, 20 parts, among them J1 Test, J2 MPU

Commit message: Added version 4 to divide in 3 boards
Parts:
- added H1, H3: STAND-OFF, SparkFun-Electromechanical:STAND-OFF
Routing:
- net GND: track 23.6 -> 24.3 mm
